Commit message: basic robot spawn in gazebo

File: ros2_ws/src/rov_sim/description/hydrodynamics.xacro (robot description, xacro)
@@ -49,22 +49,4 @@
             <nRR>-0.1857</nRR>-->
         </plugin>
-        <!-- NOT CONSIDERING AIR -->
-        <!-- <plugin
-            filename="gz-sim-buoyancy-system"
-            name="gz::sim::systems::Buoyancy">
-            <uniform_fluid_density>1000</uniform_fluid_density>
-        </plugin> -->
-        <!-- AIR DYNAMICS ABOVE WATER -->
-        <plugin
-            filename="gz-sim-buoyancy-system"
-            name="gz::sim::systems::Buoyancy">
-            <graded_buoyancy>
-                <default_density>1000</default_density>
-                <density_change>
-                <above_depth>0</above_depth>
-                <density>1</density>
-                </density_change>
-            </graded_buoyancy>
-        </plugin>
     </gazebo>
 </robot>

File: ros2_ws/src/rov_sim/description/robot.urdf.xacro (robot description, xacro)
@@ -1,5 +1,5 @@
 <?xml version="1.0"?>
 <robot xmlns:xacro="http://www.ros.org/wiki/xacro" name="robot">
-    <xacro:arg name="namespace" default="hi"/>
+    <xacro:arg name="namespace" default=""/>
     <xacro:arg name="simulation" default="true"/>
     <xacro:arg name="density" default="1000"/>
@@ -19,5 +19,7 @@
     <xacro:property name="z_cog" value="${-buoyant_correction*z_size}"/>
     <!-- Include the thruster Xacro file -->
-    <xacro:include filename="inertial_macros.xacro"/>
+    <xacro:include filename="$(find rov_sim)/description/inertial_macros.xacro"/>
+    <xacro:include filename="$(find rov_sim)/description/hydrodynamics.xacro"/>
+    <xacro:include filename="$(find rov_sim)/description/thruster.xacro"/>
     <link name="${ns}/base_link">
     </link>
@@ -36,15 +38,25 @@
         </visual>
         <collision>
-            <origin xyz="0 0 0" rpy="0 0 0"/>
+            <origin xyz="0 0 ${z_cob}" rpy="0 0 0"/>
             <geometry>
-                <box size="0.5 0.6 0.4"/>
+                <box size="${x_size*buoyant_correction} ${y_size*buoyant_correction} ${z_size*buoyant_correction}"/>
             </geometry>
         </collision>
-        <xacro:inertial_box mass="0.5" x="0.5" y="0.6" z="0.4">
-            <origin xyz="0 0 0" rpy="0 0 0"/>
-        </xacro:inertial_box>
+        <inertial>
+            <mass value="${mass}"/>
+            <origin xyz="0 0 ${z_cog}"/>
+            <!-- BlueROV2 values from "Model Predictive Control for the BlueROV2",
+                Emil Már Einarsson, Andris Lipenitis, Master thesis, 2020
+                for now make Ignition crash?-->
+            <!--         <inertia ixx="0.21" ixy="0.00" ixz="0.00" iyy="0.245" iyz="0.00" izz="0.245"/> -->
+            <inertia ixx="5.2539" ixy="0.0144" ixz="0.3341" iyy="7.9420" iyz="0.026" izz="6.9123"/>
+                <!-- Perfect rectangle -->
+            <!--        <inertia
+            ixx="${mass/12*(y_size*y_size+z_size*z_size)}" ixy="0.0" ixz="0.0"
+            iyy="${mass/12*(x_size*x_size + z_size*z_size)}" iyz="0.0"
+            izz="${mass/12*(x_size*x_size + y_size*y_size)}" />-->
+        </inertial>
     </link>
     <!-- Add multiple thrusters with different positions and orientations -->
-    <xacro:include filename="thruster.xacro"/>
     <xacro:thruster thruster_id="0" dir="CW" parent="chassis">
         <origin xyz="0.2 0.2 0.07" rpy="0 ${pi/4} ${pi/2}" />
@@ -65,8 +77,8 @@
         <origin xyz="-0.2 -0.2 -0.07" rpy="0 -${pi/4} -${pi/2}" />
     </xacro:thruster>
-    <xacro:include filename="stereo_camera.xacro"/>
-    <xacro:stereo_camera parent="chassis">
+    <!-- <xacro:include filename="stereo_camera.xacro"/> -->
+    <!-- <xacro:stereo_camera parent="chassis">
         <origin xyz="0.3 0 0" rpy="0 0 0" />
-    </xacro:stereo_camera>
+    </xacro:stereo_camera> -->
     <!-- <xacro:include filename="imu.xacro"/> -->
     <!-- <xacro:include filename="depth_sensor.xacro"/> -->

File: ros2_ws/src/rov_sim/description/stereo_camera.xacro (robot description, xacro)
@@ -12,5 +12,4 @@
                     <box size="0.010 0.03 0.03"/>
                 </geometry>
-                <material name="red"/>
             </visual>
         </link>

File: ros2_ws/src/rov_sim/description/thruster.xacro (robot description, xacro)
@@ -1,8 +1,8 @@
 <?xml version="1.0"?>
 <robot xmlns:xacro="http://www.ros.org/wiki/xacro">
-    <xacro:property name="prop_mesh_cw" value="package://rov_sim/meshes/T200_cw.dae"/>
-    <xacro:property name="prop_mesh_ccw" value="package://rov_sim/meshes/T200_ccw.dae"/>
-    <xacro:property name="prop_r" value="0.05"/>
-    <xacro:property name="prop_l" value="0.035"/>
+    <xacro:property name="prop_mesh_cw" value="file://$(find rov_sim)/meshes/T200_cw.dae"/>
+    <xacro:property name="prop_mesh_ccw" value="file://$(find rov_sim)/meshes/T200_ccw.dae"/>
+    <xacro:property name="prop_r" value="0.038"/>
+    <xacro:property name="prop_l" value="0.0508"/>
     <!--  Thruster macro: joint + link + plugin -->
     <xacro:macro name="thruster" params="thruster_id dir parent *origin">
@@ -19,5 +19,5 @@
             </visual>
             <!-- <collision>
-                    <origin rpy="0 ${PI/2} 0"/>
+                    <origin rpy="0 ${pi/2} 0"/>
                 <geometry>
                     <cylinder length="${prop_l}" radius="${prop_r}"/>
@@ -35,7 +35,7 @@
         <!-- Joint between thruster link and vehicle base link -->
         <joint name="thruster${thruster_id}" type="continuous">
+            <xacro:insert_block name="origin" />
             <parent link="${ns}/${parent}" />
             <child link="${ns}/thruster${thruster_id}" />
-            <xacro:insert_block name="origin" />
             <xacro:if value="${dir == 'CW'}">
                 <axis xyz="1 0 0" />
@@ -44,8 +44,8 @@
                 <axis xyz="-1 0 0" />
             </xacro:if>
-            <limits effort="-1" velocity="-1"/>
+            <!-- <limits effort="-1" velocity="-1"/> -->
         </joint>
     <!-- ignition topic is /model/{ns}/joint/{joint_name}/cmd_pos -->
-    <xacro:if value="$(arg simulation)">
+    <!-- <xacro:if value="$(arg simulation)"> -->
         <gazebo>
             <plugin
@@ -58,11 +58,11 @@
                 <fluid_density>${density}</fluid_density>
                 <propeller_diameter>${2*prop_r}</propeller_diameter>
-                <velocity_control>true</velocity_control>
+                <velocity_control>false</velocity_control>
                 <use_angvel_cmd>false</use_angvel_cmd>
-                <max_thrust_cmd>40</max_thrust_cmd>
-                <min_thrust_cmd>-40</min_thrust_cmd>
+                <max_thrust_cmd>51.48491</max_thrust_cmd>
+                <min_thrust_cmd>-40.2073</min_thrust_cmd>
             </plugin>
         </gazebo>
-    </xacro:if>
+    <!-- </xacro:if> -->
     </xacro:macro>
 </robot>
