Commit message: urdf

File: ros2_ws/src/rov_sim/description/robot.urdf.xacro (robot description, xacro)
@@ -65,3 +65,9 @@
         <origin xyz="-0.2 -0.2 -0.07" rpy="0 -${pi/4} -${pi/2}" />
     </xacro:thruster>
+    <xacro:include filename="stereo_camera.xacro"/>
+    <xacro:stereo_camera parent="chassis">
+        <origin xyz="0.3 0 0" rpy="0 0 0" />
+    </xacro:stereo_camera>
+    <!-- <xacro:include filename="imu.xacro"/> -->
+    <!-- <xacro:include filename="depth_sensor.xacro"/> -->
 </robot>

Commit message: add simulated depth and gps node, imu

File: ros2_ws/src/rov_sim/description/robot.urdf.xacro (robot description, xacro)
@@ -1,5 +1,5 @@
 <?xml version="1.0"?>
 <robot xmlns:xacro="http://www.ros.org/wiki/xacro" name="robot">
-    <xacro:arg name="namespace" default=""/>
+    <xacro:arg name="namespace" default="isopod"/>
     <xacro:arg name="simulation" default="true"/>
     <xacro:arg name="density" default="1000"/>
@@ -22,8 +22,10 @@
     <xacro:include filename="$(find rov_sim)/description/hydrodynamics.xacro"/>
     <xacro:include filename="$(find rov_sim)/description/thruster.xacro"/>
+    <xacro:include filename="$(find rov_sim)/description/sensors/imu.xacro"/>
+    <xacro:include filename="$(find rov_sim)/description/sensors/depth_sensor.xacro"/>
     <link name="${ns}/base_link">
     </link>
     <!-- Define the base link -->
-    <joint name="chassis_joint" type="fixed">
+    <joint name="${ns}/chassis_joint" type="fixed">
         <parent link="${ns}/base_link"/>
         <child link="${ns}/chassis"/>
@@ -77,14 +79,11 @@
         <origin xyz="-0.2 -0.2 -0.07" rpy="0 -${pi/4} -${pi/2}" />
     </xacro:thruster>
-    <!-- <xacro:include filename="stereo_camera.xacro"/> -->
-    <!-- <xacro:stereo_camera parent="chassis">
-        <origin xyz="0.3 0 0" rpy="0 0 0" />
-    </xacro:stereo_camera> -->
-    <!-- <xacro:include filename="imu.xacro"/> -->
-    <!-- <xacro:include filename="depth_sensor.xacro"/> -->
     <!-- other Gazebo plugins -->
     <xacro:if value="$(arg simulation)">
         <gazebo>
-            <plugin filename="gz-sim-joint-state-publisher-system" name="gz::sim::systems::JointStatePublisher"/>
+            <plugin
+                filename="gz-sim-joint-state-publisher-system"
+                name="gz::sim::systems::JointStatePublisher">
+            </plugin>
             <plugin
                 filename="gz-sim-odometry-publisher-system"
@@ -94,4 +93,5 @@
                 <robot_base_frame>${ns}/base_link</robot_base_frame>
                 <odom_publish_frequency>20</odom_publish_frequency>
+                <!-- <odom_topic>${ns}/odometry</odom_topic> -->
                 <dimensions>3</dimensions>
             </plugin>

File: ros2_ws/src/rov_sim/description/sensors/depth_sensor.xacro (robot description, xacro)
@@ -1,5 +1,21 @@
 <?xml version="1.0"?>
 <robot xmlns:xacro="http://www.ros.org/wiki/xacro" >
-    <xacro:macro name="depth_sensor" params="parent *origin">
+    <xacro:macro name="depth_sensor" params="name parent *origin">
+        <link name="${ns}/${name}">
+            <!-- <visual>
+                <geometry>
+                    <mesh filename="${prop_mesh_cw}"/>
+                </geometry>
+            </visual> -->
+        </link>
+        <!-- Joint between thruster link and vehicle base link -->
+        <joint name="${ns}/${name}_joint" type="fixed">
+            <xacro:insert_block name="origin" />
+            <parent link="${ns}/${parent}" />
+            <child link="${ns}/${name}" />
+        </joint>
     </xacro:macro>
+    <xacro:depth_sensor name="Bar30" parent="chassis">
+        <origin xyz="0 0 0" rpy="0 0 0"/>
+    </xacro:depth_sensor>
 </robot>

File: ros2_ws/src/rov_sim/description/sensors/imu.xacro (robot description, xacro)
@@ -1,5 +1,133 @@
 <?xml version="1.0"?>
 <robot xmlns:xacro="http://www.ros.org/wiki/xacro" >
-    <xacro:macro name="imu" params="parent *origin">
+    <xacro:macro name="imu" params="name parent *origin">
+        <link name="${ns}/${name}"/>
+        <gazebo reference="${ns}/${name}">
+        <sensor name="${name}" type="imu">
+                <always_on>1</always_on>
+                <update_rate>10</update_rate>
+                <visualize>true</visualize>
+                <topic>${ns}/${name}</topic>
+                <gz_frame_id>${ns}/${name}</gz_frame_id>
+        <imu>
+            <orientation>
+            <x>
+                <noise type="gaussian">
+                <mean>0</mean>
+                <stddev>0.009</stddev>
+                <bias_mean>0.00075</bias_mean>
+                <bias_stddev>0.005</bias_stddev>
+                <dynamic_bias_stddev>0.00002</dynamic_bias_stddev>
+                <dynamic_bias_correlation_time>400.0</dynamic_bias_correlation_time>
+                <precision>0.00025</precision>
+                </noise>
+            </x>
+            <y>
+                <noise type="gaussian">
+                <mean>0</mean>
+                <stddev>0.009</stddev>
+                <bias_mean>0.00075</bias_mean>
+                <bias_stddev>0.005</bias_stddev>
+                <dynamic_bias_stddev>0.00002</dynamic_bias_stddev>
+                <dynamic_bias_correlation_time>400.0</dynamic_bias_correlation_time>
+                <precision>0.00025</precision>
+                </noise>
+            </y>
+            <z>
+                <noise type="gaussian">
+                <mean>0</mean>
+                <stddev>0.009</stddev>
+                <bias_mean>0.00075</bias_mean>
+                <bias_stddev>0.005</bias_stddev>
+                <dynamic_bias_stddev>0.00002</dynamic_bias_stddev>
+                <dynamic_bias_correlation_time>400.0</dynamic_bias_correlation_time>
+                <precision>0.00025</precision>
+                </noise>
+            </z>
+            </orientation>
+            <angular_velocity>
+            <x>
+                <noise type="gaussian">
+                <mean>0</mean>
+                <stddev>0.009</stddev>
+                <bias_mean>0.00075</bias_mean>
+                <bias_stddev>0.005</bias_stddev>
+                <dynamic_bias_stddev>0.00002</dynamic_bias_stddev>
+                <dynamic_bias_correlation_time>400.0</dynamic_bias_correlation_time>
+                <precision>0.00025</precision>
+                </noise>
+            </x>
+            <y>
+                <noise type="gaussian">
+                <mean>0</mean>
+                <stddev>0.009</stddev>
+                <bias_mean>0.00075</bias_mean>
+                <bias_stddev>0.005</bias_stddev>
+                <dynamic_bias_stddev>0.00002</dynamic_bias_stddev>
+                <dynamic_bias_correlation_time>400.0</dynamic_bias_correlation_time>
+                <precision>0.00025</precision>
+                </noise>
+            </y>
+            <z>
+                <noise type="gaussian">
+                <mean>0</mean>
+                <stddev>0.009</stddev>
+                <bias_mean>0.00075</bias_mean>
+                <bias_stddev>0.005</bias_stddev>
+                <dynamic_bias_stddev>0.00002</dynamic_bias_stddev>
+                <dynamic_bias_correlation_time>400.0</dynamic_bias_correlation_time>
+                <precision>0.00025</precision>
+                </noise>
+            </z>
+            </angular_velocity>
+            <linear_acceleration>
+            <x>
+                <noise type="gaussian">
+                <mean>0</mean>
+                <stddev>0.021</stddev>
+                <bias_mean>0.05</bias_mean>
+                <bias_stddev>0.0075</bias_stddev>
+                <dynamic_bias_stddev>0.000375</dynamic_bias_stddev>
+                <dynamic_bias_correlation_time>175.0</dynamic_bias_correlation_time>
+                <precision>0.005</precision>
+                </noise>
+            </x>
+            <y>
+                <noise type="gaussian">
+                <mean>0</mean>
+                <stddev>0.021</stddev>
+                <bias_mean>0.05</bias_mean>
+                <bias_stddev>0.0075</bias_stddev>
+                <dynamic_bias_stddev>0.000375</dynamic_bias_stddev>
+                <dynamic_bias_correlation_time>175.0</dynamic_bias_correlation_time>
+                <precision>0.005</precision>
+                </noise>
+            </y>
+            <z>
+                <noise type="gaussian">
+                <mean>0</mean>
+                <stddev>0.021</stddev>
+                <bias_mean>0.05</bias_mean>
+                <bias_stddev>0.0075</bias_stddev>
+                <dynamic_bias_stddev>0.000375</dynamic_bias_stddev>
+                <dynamic_bias_correlation_time>175.0</dynamic_bias_correlation_time>
+                <precision>0.005</precision>
+                </noise>
+            </z>
+            </linear_acceleration>
+            <orientation_reference_frame>
+            <localization>ENU</localization>
+            </orientation_reference_frame>
+        </imu>
+            </sensor>
+        </gazebo>
+        <joint name="${ns}/{name}_joint" type="fixed">
+            <xacro:insert_block name="origin"/>
+            <parent link="${ns}/${parent}"/>
+            <child link="${ns}/${name}"/>
+        </joint>
     </xacro:macro>
+    <xacro:imu name="imu" parent="chassis">
+        <origin xyz="0 0 0" rpy="0 0 0"/>
+    </xacro:imu>
 </robot>

File: ros2_ws/src/rov_sim/description/sensors/stereo_camera.xacro (robot description, xacro)
@@ -1,11 +1,11 @@
 <?xml version="1.0"?>
 <robot xmlns:xacro="http://www.ros.org/wiki/xacro" >
-    <xacro:macro name="stereo_camera" params="parent *origin">
-        <joint name="camera_joint" type="fixed">
+    <xacro:macro name="camera" params="name parent *origin">
+        <joint name="camera_joint" type="revolute">
             <parent link="${ns}/${parent}"/>
-            <child link="camera_link"/>
+            <child link="${ns}/${name}_link"/>
             <xacro:insert_block name="origin" />
         </joint>
-        <link name="camera_link">
+        <link name="${ns}/${name}">
             <visual>
                 <geometry>

File: ros2_ws/src/rov_sim/description/thruster.xacro (robot description, xacro)
@@ -34,5 +34,5 @@
         </link>
         <!-- Joint between thruster link and vehicle base link -->
-        <joint name="thruster${thruster_id}" type="continuous">
+        <joint name="${ns}/thruster${thruster_id}_joint" type="continuous">
             <xacro:insert_block name="origin" />
             <parent link="${ns}/${parent}" />
@@ -52,7 +52,6 @@
                 filename="gz-sim-thruster-system"
                 name="gz::sim::systems::Thruster">
-                <namespace>${ns}</namespace>
-                <joint_name>thruster${thruster_id}</joint_name>
-                <topic>${ns}/thruster${thruster_id}/cmd</topic>
+                <joint_name>${ns}/thruster${thruster_id}_joint</joint_name>
+                <topic>thruster${thruster_id}/cmd</topic>
                 <thrust_coefficient>0.011</thrust_coefficient>
                 <fluid_density>${density}</fluid_density>

Commit message: wrench to sim works, need to fix thruster direction

File: ros2_ws/src/rov_sim/description/robot.urdf.xacro (robot description, xacro)
@@ -61,21 +61,21 @@
     </link>
     <!-- Add multiple thrusters with different positions and orientations -->
-    <xacro:thruster thruster_id="0" dir="CW" parent="chassis">
-        <origin xyz="0.2 0.2 0.07" rpy="0 ${pi/4} ${pi/2}" />
+    <xacro:thruster thruster_id="0" dir="CCW" parent="chassis">
+        <origin xyz="0.151 0.10815 0.09222" rpy="0 ${pi/4} ${pi/2}" />
     </xacro:thruster>
     <xacro:thruster thruster_id="1" dir="CCW" parent="chassis">
-        <origin xyz="0 0.25 0" rpy="${pi} -${pi} 0" />
+        <origin xyz="-0.01506 0.161 0" rpy="${pi} -${pi} 0" />
     </xacro:thruster>
     <xacro:thruster thruster_id="2" dir="CW" parent="chassis">
-        <origin xyz="-0.2 0.2 -0.07" rpy="0 -${pi/4} ${pi/2}" />
+        <origin xyz="-0.134 0.10815 -0.09222" rpy="0 -${pi/4} ${pi/2}" />
     </xacro:thruster>
-    <xacro:thruster thruster_id="3" dir="CCW" parent="chassis">
-        <origin xyz="0.2 -0.2 0.07" rpy="0 ${pi/4} -${pi/2}" />
+    <xacro:thruster thruster_id="3" dir="CW" parent="chassis">
+        <origin xyz="0.151 -0.10815 0.09222" rpy="0 ${pi/4} -${pi/2}" />
     </xacro:thruster>
     <xacro:thruster thruster_id="4" dir="CW" parent="chassis">
-        <origin xyz="0 -0.25 0" rpy="${pi} -${pi} 0" />
+        <origin xyz="-0.01506 -0.161 0" rpy="${pi} -${pi} 0" />
     </xacro:thruster>
     <xacro:thruster thruster_id="5" dir="CCW" parent="chassis">
-        <origin xyz="-0.2 -0.2 -0.07" rpy="0 -${pi/4} -${pi/2}" />
+        <origin xyz="-0.134 -0.10815 -0.09222" rpy="0 -${pi/4} -${pi/2}" />
     </xacro:thruster>
     <!-- other Gazebo plugins -->

File: ros2_ws/src/rov_sim/description/thruster.xacro (robot description, xacro)
@@ -18,10 +18,4 @@
                 </geometry>
             </visual>
-            <!-- <collision>
-                    <origin rpy="0 ${pi/2} 0"/>
-                <geometry>
-                    <cylinder length="${prop_l}" radius="${prop_r}"/>
-                </geometry>
-            </collision> -->
             <inertial>
                 <!-- thruster axis is X -->
@@ -46,5 +40,4 @@
             <limits effort="51.48491"/>
         </joint>
-    <!-- ignition topic is /model/{ns}/joint/{joint_name}/cmd_pos -->
     <!-- <xacro:if value="$(arg simulation)"> -->
         <gazebo>
