Commit message: fixed transform, removed ns, cov not published

File: ros2_ws/src/rov_sim/description/robot.urdf.xacro (robot description, xacro)
@@ -1,5 +1,5 @@
 <?xml version="1.0"?>
 <robot xmlns:xacro="http://www.ros.org/wiki/xacro" name="robot">
-    <xacro:arg name="namespace" default="isopod"/>
+    <xacro:arg name="namespace" default=""/>
     <xacro:arg name="simulation" default="true"/>
     <xacro:arg name="density" default="1000"/>
@@ -24,4 +24,5 @@
     <xacro:include filename="$(find rov_sim)/description/sensors/imu.xacro"/>
     <xacro:include filename="$(find rov_sim)/description/sensors/depth_sensor.xacro"/>
+    <xacro:include filename="$(find rov_sim)/description/sensors/gps.xacro"/>
     <link name="${ns}/base_link">
     </link>

File: ros2_ws/src/rov_sim/description/sensors/gps.xacro (robot description, xacro)
@@ -3,9 +3,4 @@
     <xacro:macro name="gps_sensor" params="name parent *origin">
         <link name="${ns}/${name}">
-            <!-- <visual>
-                <geometry>
-                    <mesh filename="${prop_mesh_cw}"/>
-                </geometry>
-            </visual> -->
         </link>
         <!-- Joint between thruster link and vehicle base link -->
@@ -16,16 +11,52 @@
         </joint>
         <gazebo reference="${ns}/${name}">
-            <plugin
-                filename="gz-sim-navsat-system"
-                name="gz::sim::systems::NavSat">
-            </plugin>
-            <sensor name="navsat_sensor" type="navsat">
+            <sensor name="${name}" type="navsat">
                 <always_on>1</always_on>
                 <update_rate>30</update_rate>
+                <topic>${ns}/${name}</topic>
+                <gz_frame_id>${ns}/${name}</gz_frame_id>
+                <gps>
+                    <position_sensing>
+                        <horizontal>
+                        <noise type="gaussian">
+                            <mean>0.0</mean>
+                            <stddev>0.1</stddev>
+                            <bias_mean>0.0</bias_mean>
+                            <bias_stddev>0.0</bias_stddev>
+                        </noise>
+                        </horizontal>
+                        <vertical>
+                        <noise type="gaussian">
+                            <mean>0.0</mean>
+                            <stddev>0.1</stddev>
+                            <bias_mean>0.0</bias_mean>
+                            <bias_stddev>0.0</bias_stddev>
+                        </noise>
+                        </vertical>
+                    </position_sensing>
+                    <velocity_sensing>
+                        <horizontal>
+                        <noise type="gaussian">
+                            <mean>0.0</mean>
+                            <stddev>0.2</stddev>
+                            <bias_mean>0.0</bias_mean>
+                            <bias_stddev>0.0</bias_stddev>
+                        </noise>
+                        </horizontal>
+                        <vertical>
+                        <noise type="gaussian">
+                            <mean>0.0</mean>
+                            <stddev>0.2</stddev>
+                            <bias_mean>0.0</bias_mean>
+                            <bias_stddev>0.0</bias_stddev>
+                        </noise>
+                        </vertical>
+                    </velocity_sensing>
+                </gps>
             </sensor>
         </gazebo>
     </xacro:macro>
-    <xacro:depth_sensor name="Bar30" parent="chassis">
-        <origin xyz="0 0 0" rpy="0 0 0"/>
-    </xacro:depth_sensor>
+    <xacro:gps_sensor name="gps" parent="chassis">
+        <origin xyz="0 0 0.010" rpy="0 0 0"/>
+    </xacro:gps_sensor>
 </robot>

File: ros2_ws/src/rov_sim/description/sensors/imu.xacro (robot description, xacro)
@@ -11,111 +11,77 @@
                 <gz_frame_id>${ns}/${name}</gz_frame_id>
                 <imu>
-                    <orientation>
-                    <x>
-                        <noise type="gaussian">
-                        <mean>0</mean>
-                        <stddev>0.009</stddev>
-                        <bias_mean>0.00075</bias_mean>
-                        <bias_stddev>0.005</bias_stddev>
-                        <dynamic_bias_stddev>0.00002</dynamic_bias_stddev>
-                        <dynamic_bias_correlation_time>400.0</dynamic_bias_correlation_time>
-                        <precision>0.00025</precision>
-                        </noise>
-                    </x>
-                    <y>
-                        <noise type="gaussian">
-                        <mean>0</mean>
-                        <stddev>0.009</stddev>
-                        <bias_mean>0.00075</bias_mean>
-                        <bias_stddev>0.005</bias_stddev>
-                        <dynamic_bias_stddev>0.00002</dynamic_bias_stddev>
-                        <dynamic_bias_correlation_time>400.0</dynamic_bias_correlation_time>
-                        <precision>0.00025</precision>
-                        </noise>
-                    </y>
-                    <z>
-                        <noise type="gaussian">
-                        <mean>0</mean>
-                        <stddev>0.009</stddev>
-                        <bias_mean>0.00075</bias_mean>
-                        <bias_stddev>0.005</bias_stddev>
-                        <dynamic_bias_stddev>0.00002</dynamic_bias_stddev>
-                        <dynamic_bias_correlation_time>400.0</dynamic_bias_correlation_time>
-                        <precision>0.00025</precision>
-                        </noise>
-                    </z>
-                    </orientation>
+                    <enable_orientation>true</enable_orientation>
                     <angular_velocity>
-                    <x>
-                        <noise type="gaussian">
-                        <mean>0</mean>
-                        <stddev>0.009</stddev>
-                        <bias_mean>0.00075</bias_mean>
-                        <bias_stddev>0.005</bias_stddev>
-                        <dynamic_bias_stddev>0.00002</dynamic_bias_stddev>
-                        <dynamic_bias_correlation_time>400.0</dynamic_bias_correlation_time>
-                        <precision>0.00025</precision>
-                        </noise>
-                    </x>
-                    <y>
-                        <noise type="gaussian">
-                        <mean>0</mean>
-                        <stddev>0.009</stddev>
-                        <bias_mean>0.00075</bias_mean>
-                        <bias_stddev>0.005</bias_stddev>
-                        <dynamic_bias_stddev>0.00002</dynamic_bias_stddev>
-                        <dynamic_bias_correlation_time>400.0</dynamic_bias_correlation_time>
-                        <precision>0.00025</precision>
-                        </noise>
-                    </y>
-                    <z>
-                        <noise type="gaussian">
-                        <mean>0</mean>
-                        <stddev>0.009</stddev>
-                        <bias_mean>0.00075</bias_mean>
-                        <bias_stddev>0.005</bias_stddev>
-                        <dynamic_bias_stddev>0.00002</dynamic_bias_stddev>
-                        <dynamic_bias_correlation_time>400.0</dynamic_bias_correlation_time>
-                        <precision>0.00025</precision>
-                        </noise>
-                    </z>
+                        <x>
+                            <noise type="gaussian">
+                            <mean>0</mean>
+                            <stddev>0.009</stddev>
+                            <bias_mean>0.00075</bias_mean>
+                            <bias_stddev>0.005</bias_stddev>
+                            <dynamic_bias_stddev>0.00002</dynamic_bias_stddev>
+                            <dynamic_bias_correlation_time>400.0</dynamic_bias_correlation_time>
+                            <precision>0.00025</precision>
+                            </noise>
+                        </x>
+                        <y>
+                            <noise type="gaussian">
+                            <mean>0</mean>
+                            <stddev>0.009</stddev>
+                            <bias_mean>0.00075</bias_mean>
+                            <bias_stddev>0.005</bias_stddev>
+                            <dynamic_bias_stddev>0.00002</dynamic_bias_stddev>
+                            <dynamic_bias_correlation_time>400.0</dynamic_bias_correlation_time>
+                            <precision>0.00025</precision>
+                            </noise>
+                        </y>
+                        <z>
+                            <noise type="gaussian">
+                            <mean>0</mean>
+                            <stddev>0.009</stddev>
+                            <bias_mean>0.00075</bias_mean>
+                            <bias_stddev>0.005</bias_stddev>
+                            <dynamic_bias_stddev>0.00002</dynamic_bias_stddev>
+                            <dynamic_bias_correlation_time>400.0</dynamic_bias_correlation_time>
+                            <precision>0.00025</precision>
+                            </noise>
+                        </z>
                     </angular_velocity>
                     <linear_acceleration>
-                    <x>
-                        <noise type="gaussian">
-                        <mean>0</mean>
-                        <stddev>0.021</stddev>
-                        <bias_mean>0.05</bias_mean>
-                        <bias_stddev>0.0075</bias_stddev>
-                        <dynamic_bias_stddev>0.000375</dynamic_bias_stddev>
-                        <dynamic_bias_correlation_time>175.0</dynamic_bias_correlation_time>
-                        <precision>0.005</precision>
-                        </noise>
-                    </x>
-                    <y>
-                        <noise type="gaussian">
-                        <mean>0</mean>
-                        <stddev>0.021</stddev>
-                        <bias_mean>0.05</bias_mean>
-                        <bias_stddev>0.0075</bias_stddev>
-                        <dynamic_bias_stddev>0.000375</dynamic_bias_stddev>
-                        <dynamic_bias_correlation_time>175.0</dynamic_bias_correlation_time>
-                        <precision>0.005</precision>
-                        </noise>
-                    </y>
-                    <z>
-                        <noise type="gaussian">
-                        <mean>0</mean>
-                        <stddev>0.021</stddev>
-                        <bias_mean>0.05</bias_mean>
-                        <bias_stddev>0.0075</bias_stddev>
-                        <dynamic_bias_stddev>0.000375</dynamic_bias_stddev>
-                        <dynamic_bias_correlation_time>175.0</dynamic_bias_correlation_time>
-                        <precision>0.005</precision>
-                        </noise>
-                    </z>
+                        <x>
+                            <noise type="gaussian">
+                            <mean>0</mean>
+                            <stddev>0.021</stddev>
+                            <bias_mean>0.05</bias_mean>
+                            <bias_stddev>0.0075</bias_stddev>
+                            <dynamic_bias_stddev>0.000375</dynamic_bias_stddev>
+                            <dynamic_bias_correlation_time>175.0</dynamic_bias_correlation_time>
+                            <precision>0.005</precision>
+                            </noise>
+                        </x>
+                        <y>
+                            <noise type="gaussian">
+                            <mean>0</mean>
+                            <stddev>0.021</stddev>
+                            <bias_mean>0.05</bias_mean>
+                            <bias_stddev>0.0075</bias_stddev>
+                            <dynamic_bias_stddev>0.000375</dynamic_bias_stddev>
+                            <dynamic_bias_correlation_time>175.0</dynamic_bias_correlation_time>
+                            <precision>0.005</precision>
+                            </noise>
+                        </y>
+                        <z>
+                            <noise type="gaussian">
+                            <mean>0</mean>
+                            <stddev>0.021</stddev>
+                            <bias_mean>0.05</bias_mean>
+                            <bias_stddev>0.0075</bias_stddev>
+                            <dynamic_bias_stddev>0.000375</dynamic_bias_stddev>
+                            <dynamic_bias_correlation_time>175.0</dynamic_bias_correlation_time>
+                            <precision>0.005</precision>
+                            </noise>
+                        </z>
                     </linear_acceleration>
                     <orientation_reference_frame>
-                    <localization>ENU</localization>
+                        <localization>ENU</localization>
                     </orientation_reference_frame>
                 </imu>

File: ros2_ws/src/rov_sim/description/thruster.xacro (robot description, xacro)
@@ -38,5 +38,5 @@
                 <axis xyz="-1 0 0" />
             </xacro:if>
-            <limits effort="51.48491"/>
+            <limits effort="-1" velocity="-1"/>
         </joint>
     <!-- <xacro:if value="$(arg simulation)"> -->
@@ -47,9 +47,11 @@
                 <joint_name>${ns}/thruster${thruster_id}_joint</joint_name>
                 <topic>thruster${thruster_id}/cmd</topic>
-                <thrust_coefficient>0.011</thrust_coefficient>
+                <!-- <use_angvel_cmd>true</use_angvel_cmd> -->
+                <!-- <velocity_control>false</velocity_control> -->
+                <!-- <thrust_coefficient>80.2073</thrust_coefficient> -->
                 <fluid_density>${density}</fluid_density>
                 <propeller_diameter>${2*prop_r}</propeller_diameter>
-                <velocity_control>false</velocity_control>
-                <use_angvel_cmd>false</use_angvel_cmd>
+                <!-- <max_thrust_cmd>1.2805</max_thrust_cmd> -->
+                <!-- <min_thrust_cmd>-1.0</min_thrust_cmd> -->
                 <max_thrust_cmd>51.48491</max_thrust_cmd>
                 <min_thrust_cmd>-40.2073</min_thrust_cmd>
