Commit message: reorganize

File: ros2_ws/src/rov/rov_control/description/ros2_control.xacro (robot description, xacro)
@@ -1,57 +1,107 @@
 <?xml version="1.0"?>
 <robot xmlns:xacro="http://www.ros.org/wiki/xacro">
-    <ros2_control name="GazeboSystem" type="system">
+    <link name="x_link">
+    </link>
+    <link name="y_link">
+    </link>
+    <link name="z_link">
+    </link>
+    <link name="rx_link">
+    </link>
+    <link name="ry_link">
+    </link>
+    <link name="rz_link">
+    </link>
+    <!-- Cartesian Joints -->
+    <joint name="x"
+            type="continuous">
+    <parent link="base_link" />
+    <child link="x_link" />
+    </joint>
+    <joint name="y"
+            type="continuous">
+    <parent link="base_link" />
+    <child link="y_link" />
+    </joint>
+    <joint name="z"
+            type="continuous">
+    <parent link="base_link" />
+    <child link="z_link" />
+    </joint>
+    <joint name="rx"
+            type="continuous">
+    <parent link="base_link" />
+    <child link="rx_link" />
+    </joint>
+    <joint name="ry"
+            type="continuous">
+    <parent link="base_link" />
+    <child link="ry_link" />
+    </joint>
+    <joint name="rz"
+            type="continuous">
+    <parent link="base_link" />
+    <child link="rz_link" />
+    </joint>
+    <ros2_control name="demo_hardware"
+                type="system">
         <hardware>
-            <plugin>gazebo_ros2_control/GazeboSystem</plugin>
-            <joint name="x_acceleration">
-                <command_interface name="effort">
-                    <param name="min">-10.0</param>
-                    <param name="max">10.0</param>
-                </command_interface>
-                <state_interface name="acceleration"/>
-            </joint>
-            <joint name="y_acceleration">
-                <command_interface name="effort">
-                    <param name="min">-10.0</param>
-                    <param name="max">10.0</param>
-                </command_interface>
-                <state_interface name="acceleration"/>
-            </joint>
-            <joint name="z_position">
-                <command_interface name="position">
-                </command_interface>
-                <state_interface name="acceleration"/>
-                <state_interface name="position"/>
-            </joint>
-            <joint name="roll">
-                <command_interface name="position">
-                    <param name="min">-1.0</param>
-                    <param name="max">1.0</param>
-                </command_interface>
-                <state_interface name="orientation"/>
-                <state_interface name="velocity"/>
-            </joint>
-            <joint name="pitch">
-                <command_interface name="effort">
-                    <param name="min">-1.0</param>
-                    <param name="max">1.0</param>
-                </command_interface>
-                <state_interface name="orientation"/>
-                <state_interface name="velocity"/>
-            </joint>
-            <joint name="yaw">
-                <command_interface name="effort">
-                    <param name="min">-1.0</param>
-                    <param name="max">1.0</param>
-                </command_interface>
-                <state_interface name="orientation"/>
-                <state_interface name="velocity"/>
-            </joint>
+            <plugin>mock_components/GenericSystem</plugin>
+            <param name="calculate_dynamics">false</param>
         </hardware>
+        <joint name="x">
+            <state_interface name="position">
+            <param name="initial_value">0.0</param>
+            </state_interface>
+            <state_interface name="velocity">
+            <param name="initial_value">0.0</param>
+            </state_interface>
+            <command_interface name="effort" />
+        </joint>
+        <joint name="y">
+            <state_interface name="position">
+            <param name="initial_value">0.0</param>
+            </state_interface>
+            <state_interface name="velocity">
+            <param name="initial_value">0.0</param>
+            </state_interface>
+            <command_interface name="effort" />
+        </joint>
+        <joint name="z">
+            <state_interface name="position">
+            <param name="initial_value">0.0</param>
+            </state_interface>
+            <state_interface name="velocity">
+            <param name="initial_value">0.0</param>
+            </state_interface>
+            <command_interface name="effort" />
+        </joint>
+        <joint name="rx">
+            <state_interface name="position">
+            <param name="initial_value">0.0</param>
+            </state_interface>
+            <state_interface name="velocity">
+            <param name="initial_value">0.0</param>
+            </state_interface>
+            <command_interface name="effort" />
+        </joint>
+        <joint name="ry">
+            <state_interface name="position">
+            <param name="initial_value">0.0</param>
+            </state_interface>
+            <state_interface name="velocity">
+            <param name="initial_value">0.0</param>
+            </state_interface>
+            <command_interface name="effort" />
+        </joint>
+        <joint name="rz">
+            <state_interface name="position">
+            <param name="initial_value">0.0</param>
+            </state_interface>
+            <state_interface name="velocity">
+            <param name="initial_value">0.0</param>
+            </state_interface>
+            <command_interface name="effort" />
+        </joint>
     </ros2_control>
-    <gazebo>
-        <plugin filename="libgazebo_ros2_control.so" name="gazebo_ros2_control">
-            <parameters>...to be filled in soon!...</parameters>
-        </plugin>
-    </gazebo>
 </robot>

File: ros2_ws/src/rov/rov_description/description/hydrodynamics.xacro (robot description, xacro)
@@ -6,5 +6,5 @@
             name="gz::sim::systems::Hydrodynamics">
             <!--     <density>${density}</density> -->
-            <link_name>${ns}/base_link</link_name>
+            <link_name>base_link</link_name>
             <!-- <default_current>0.05 0.03 0.0</default_current> -->
             <!-- BlueROV2 heavy values from "6-DoF Modelling and Control of a Remotely Operated Vehicle"

File: ros2_ws/src/rov/rov_description/description/robot.urdf.xacro (robot description, xacro)
@@ -1,5 +1,4 @@
 <?xml version="1.0"?>
 <robot xmlns:xacro="http://www.ros.org/wiki/xacro" name="robot">
-    <xacro:arg name="namespace" default=""/>
     <xacro:arg name="simulation" default="true"/>
     <xacro:arg name="density" default="1000"/>
@@ -19,19 +18,19 @@
     <xacro:property name="z_cog" value="${-buoyant_correction*z_size}"/>
     <!-- Include the thruster Xacro file -->
-    <xacro:include filename="$(find rov_sim)/description/inertial_macros.xacro"/>
-    <xacro:include filename="$(find rov_sim)/description/hydrodynamics.xacro"/>
-    <xacro:include filename="$(find rov_sim)/description/thruster.xacro"/>
-    <xacro:include filename="$(find rov_sim)/description/sensors/imu.xacro"/>
-    <xacro:include filename="$(find rov_sim)/description/sensors/depth_sensor.xacro"/>
-    <xacro:include filename="$(find rov_sim)/description/sensors/gps.xacro"/>
-    <link name="${ns}/base_link">
+    <xacro:include filename="$(find rov_description)/description/inertial_macros.xacro"/>
+    <xacro:include filename="$(find rov_description)/description/thruster.xacro"/>
+    <xacro:include filename="$(find rov_description)/description/sensors/imu.xacro"/>
+    <xacro:include filename="$(find rov_description)/description/sensors/depth_sensor.xacro"/>
+    <xacro:include filename="$(find rov_description)/description/sensors/gps.xacro"/>
+    <xacro:include filename="$(find rov_control)/description/ros2_control.xacro"/>
+    <link name="base_link">
     </link>
     <!-- Define the base link -->
-    <joint name="${ns}/chassis_joint" type="fixed">
-        <parent link="${ns}/base_link"/>
-        <child link="${ns}/chassis"/>
+    <joint name="chassis_joint" type="fixed">
+        <parent link="base_link"/>
+        <child link="chassis"/>
         <origin xyz="0 0 0"/>
     </joint>
-    <link name="${ns}/chassis">
+    <link name="chassis">
         <visual>
             <origin xyz="0 0 0" rpy="0 0 0"/>
@@ -80,6 +79,6 @@
         <origin xyz="-0.134 -0.10815 -0.09222" rpy="0 -${pi/4} -${pi/2}" />
     </xacro:thruster>
-    <!-- other Gazebo plugins -->
     <xacro:if value="$(arg simulation)">
+        <xacro:include filename="$(find rov_description)/description/hydrodynamics.xacro"/>
         <gazebo>
             <plugin
@@ -92,10 +91,11 @@
                 <odom_frame>world</odom_frame>
                 <dimensions>3</dimensions>
-                <robot_base_frame>${ns}/base_link</robot_base_frame>
+                <robot_base_frame>base_link</robot_base_frame>
                 <odom_publish_frequency>20</odom_publish_frequency>
-                <!-- <odom_topic>${ns}/odometry</odom_topic> -->
                 <dimensions>3</dimensions>
+                <gaussian_noise>0.5</gaussian_noise>
             </plugin>
-            <plugin
+            <!-- If you want to publish world -> base_link transform -->
+            <!-- <plugin
                 filename="gz-sim-pose-publisher-system"
                 name="gz::sim::systems::PosePublisher">
@@ -104,5 +104,5 @@
                 <publish_visual_pose>false</publish_visual_pose>
                 <publish_nested_model_pose>true</publish_nested_model_pose>
-            </plugin>
+            </plugin> -->
         </gazebo>
     </xacro:if>

File: ros2_ws/src/rov/rov_description/description/sensors/depth_sensor.xacro (robot description, xacro)
@@ -2,5 +2,5 @@
 <robot xmlns:xacro="http://www.ros.org/wiki/xacro" >
     <xacro:macro name="depth_sensor" params="name parent *origin">
-        <link name="${ns}/${name}">
+        <link name="${name}">
             <!-- <visual>
                 <geometry>
@@ -10,8 +10,8 @@
         </link>
         <!-- Joint between thruster link and vehicle base link -->
-        <joint name="${ns}/${name}_joint" type="fixed">
+        <joint name="${name}_joint" type="fixed">
             <xacro:insert_block name="origin" />
-            <parent link="${ns}/${parent}" />
-            <child link="${ns}/${name}" />
+            <parent link="${parent}" />
+            <child link="${name}" />
         </joint>
     </xacro:macro>

File: ros2_ws/src/rov/rov_description/description/sensors/stereo_camera.xacro (robot description, xacro)
@@ -3,9 +3,9 @@
     <xacro:macro name="camera" params="name parent *origin">
         <joint name="camera_joint" type="revolute">
-            <parent link="${ns}/${parent}"/>
-            <child link="${ns}/${name}_link"/>
+            <parent link="${parent}"/>
+            <child link="${name}_link"/>
             <xacro:insert_block name="origin" />
         </joint>
-        <link name="${ns}/${name}">
+        <link name="${name}">
             <visual>
                 <geometry>
@@ -48,5 +48,5 @@
                 </camera>
                 <visualize>true</visualize>
-                <topic>${ns}/image</topic>
+                <topic>image</topic>
                 <enable_metrics>false</enable_metrics>
                 <plugin name="camera_controller" filename="libgazebo_ros_camera.so">

File: ros2_ws/src/rov/rov_description/description/thruster.xacro (robot description, xacro)
@@ -1,11 +1,11 @@
 <?xml version="1.0"?>
 <robot xmlns:xacro="http://www.ros.org/wiki/xacro">
-    <xacro:property name="prop_mesh_cw" value="file://$(find rov_sim)/meshes/T200_cw.dae"/>
-    <xacro:property name="prop_mesh_ccw" value="file://$(find rov_sim)/meshes/T200_ccw.dae"/>
+    <xacro:property name="prop_mesh_cw" value="file://$(find rov_description)/meshes/T200_cw.dae"/>
+    <xacro:property name="prop_mesh_ccw" value="file://$(find rov_description)/meshes/T200_ccw.dae"/>
     <xacro:property name="prop_r" value="0.038"/>
     <xacro:property name="prop_l" value="0.0508"/>
     <!--  Thruster macro: joint + link + plugin -->
     <xacro:macro name="thruster" params="thruster_id dir parent *origin">
-        <link name="${ns}/thruster${thruster_id}">
+        <link name="thruster${thruster_id}">
             <visual>
                 <geometry>
@@ -28,8 +28,8 @@
         </link>
         <!-- Joint between thruster link and vehicle base link -->
-        <joint name="${ns}/thruster${thruster_id}_joint" type="continuous">
+        <joint name="thruster${thruster_id}_joint" type="continuous">
             <xacro:insert_block name="origin" />
-            <parent link="${ns}/${parent}" />
-            <child link="${ns}/thruster${thruster_id}" />
+            <parent link="${parent}" />
+            <child link="thruster${thruster_id}" />
             <xacro:if value="${dir == 'CW'}">
                 <axis xyz="1 0 0" />
@@ -40,10 +40,10 @@
             <limits effort="-1" velocity="-1"/>
         </joint>
-    <!-- <xacro:if value="$(arg simulation)"> -->
+    <xacro:if value="$(arg simulation)">
         <gazebo>
             <plugin
                 filename="gz-sim-thruster-system"
                 name="gz::sim::systems::Thruster">
-                <joint_name>${ns}/thruster${thruster_id}_joint</joint_name>
+                <joint_name>thruster${thruster_id}_joint</joint_name>
                 <topic>thruster${thruster_id}/cmd</topic>
                 <!-- <use_angvel_cmd>true</use_angvel_cmd> -->
@@ -58,5 +58,5 @@
             </plugin>
         </gazebo>
-    <!-- </xacro:if> -->
+    </xacro:if>
     </xacro:macro>
 </robot>

Commit message: add camera, make world blue

File: ros2_ws/src/rov/rov_control/description/ros2_control.xacro (robot description, xacro)
@@ -43,4 +43,11 @@
     <parent link="base_link" />
     <child link="rz_link" />
+    </joint>
+    <link name="control_link">
+    </link>
+    <joint name="control_joint"
+            type="floating">
+    <parent link="base_link" />
+    <child link="control_link" />
     </joint>
     <ros2_control name="demo_hardware"

File: ros2_ws/src/rov/rov_description/description/robot.urdf.xacro (robot description, xacro)
@@ -23,5 +23,6 @@
     <xacro:include filename="$(find rov_description)/description/sensors/depth_sensor.xacro"/>
     <xacro:include filename="$(find rov_description)/description/sensors/gps.xacro"/>
-    <xacro:include filename="$(find rov_control)/description/ros2_control.xacro"/>
+    <xacro:include filename="$(find rov_description)/description/sensors/camera.xacro"/>
+    <!-- <xacro:include filename="$(find rov_control)/description/ros2_control.xacro"/> -->
     <link name="base_link">
     </link>

File: ros2_ws/src/rov/rov_description/description/sensors/depth_sensor.xacro (robot description, xacro)
@@ -3,11 +3,5 @@
     <xacro:macro name="depth_sensor" params="name parent *origin">
         <link name="${name}">
-            <!-- <visual>
-                <geometry>
-                    <mesh filename="${prop_mesh_cw}"/>
-                </geometry>
-            </visual> -->
         </link>
-        <!-- Joint between thruster link and vehicle base link -->
         <joint name="${name}_joint" type="fixed">
             <xacro:insert_block name="origin" />
