Commit message: simulation cleanup

File: ros2_ws/src/rov/rov_description/description/robot.urdf.xacro (robot description, xacro)
@@ -1,27 +1,28 @@
 <?xml version="1.0"?>
 <robot xmlns:xacro="http://www.ros.org/wiki/xacro" name="robot">
-    <xacro:arg name="simulation" default="true"/>
-    <xacro:arg name="density" default="1000"/>
-    <xacro:property name="ns" value="$(arg namespace)"/>
-    <xacro:property name="density" value="$(arg density)"/>
-    <xacro:property name="x_size" value="0.40"/>
-    <xacro:property name="y_size" value="0.25"/>
-    <xacro:property name="z_size" value="0.1"/>
-    <xacro:property name="mass" value="14.8"/>
+    <xacro:arg name="simulation" default="true" />
+    <xacro:arg name="density" default="1000" />
+    <xacro:property name="ns" value="$(arg namespace)" />
+    <xacro:property name="density" value="$(arg density)" />
+    <xacro:property name="x_size" value="0.40" />
+    <xacro:property name="y_size" value="0.25" />
+    <xacro:property name="z_size" value="0.1" />
+    <xacro:property name="mass" value="14.8" />
     <!-- other props -->
-    <xacro:property name="prop_mass" value="0.07"/>
+    <xacro:property name="prop_mass" value="0.07" />
     <!-- to set correct buoyancy volume with 1 % positive factor -->
-    <xacro:property name="buoyant_correction" value="${1.01*pow((mass + 6*prop_mass)/(density*x_size*y_size*z_size), 1./3)}"/>
+    <xacro:property name="buoyant_correction"
+        value="${1.01*pow((mass + 6*prop_mass)/(density*x_size*y_size*z_size), 1./3)}" />
     <!-- Center of buoyancy -->
-    <xacro:property name="z_cob" value="${-buoyant_correction*z_size/4}"/>
+    <xacro:property name="z_cob" value="${-buoyant_correction*z_size/4}" />
     <!-- Center of gravity -->
-    <xacro:property name="z_cog" value="${-buoyant_correction*z_size}"/>
+    <xacro:property name="z_cog" value="${-buoyant_correction*z_size}" />
     <!-- Include the thruster Xacro file -->
-    <xacro:include filename="$(find rov_description)/description/inertial_macros.xacro"/>
-    <xacro:include filename="$(find rov_description)/description/thruster.xacro"/>
-    <xacro:include filename="$(find rov_description)/description/sensors/imu.xacro"/>
-    <xacro:include filename="$(find rov_description)/description/sensors/depth_sensor.xacro"/>
-    <xacro:include filename="$(find rov_description)/description/sensors/gps.xacro"/>
-    <xacro:include filename="$(find rov_description)/description/sensors/camera.xacro"/>
+    <xacro:include filename="$(find rov_description)/description/inertial_macros.xacro" />
+    <xacro:include filename="$(find rov_description)/description/thruster.xacro" />
+    <xacro:include filename="$(find rov_description)/description/sensors/imu.xacro" />
+    <xacro:include filename="$(find rov_description)/description/sensors/depth_sensor.xacro" />
+    <xacro:include filename="$(find rov_description)/description/sensors/gps.xacro" />
+    <xacro:include filename="$(find rov_description)/description/sensors/camera.xacro" />
     <!-- <xacro:include filename="$(find rov_control)/description/ros2_control.xacro"/> -->
     <link name="base_link">
@@ -29,30 +30,31 @@
     <!-- Define the base link -->
     <joint name="chassis_joint" type="fixed">
-        <parent link="base_link"/>
-        <child link="chassis"/>
-        <origin xyz="0 0 0"/>
+        <parent link="base_link" />
+        <child link="chassis" />
+        <origin xyz="0 0 0" />
     </joint>
     <link name="chassis">
         <visual>
-            <origin xyz="0 0 0" rpy="0 0 0"/>
+            <origin xyz="0 0 0" rpy="0 0 0" />
             <geometry>
-                <box size="0.3 0.3 0.05"/>
+                <box size="0.3 0.3 0.05" />
             </geometry>
         </visual>
         <collision>
-            <origin xyz="0 0 ${z_cob}" rpy="0 0 0"/>
+            <origin xyz="0 0 ${z_cob}" rpy="0 0 0" />
             <geometry>
-                <box size="${x_size*buoyant_correction} ${y_size*buoyant_correction} ${z_size*buoyant_correction}"/>
+                <box
+                    size="${x_size*buoyant_correction} ${y_size*buoyant_correction} ${z_size*buoyant_correction}" />
             </geometry>
         </collision>
         <inertial>
-            <mass value="${mass}"/>
-            <origin xyz="0 0 ${z_cog}"/>
+            <mass value="${mass}" />
+            <origin xyz="0 0 ${z_cog}" />
             <!-- BlueROV2 values from "Model Predictive Control for the BlueROV2",
                 Emil Már Einarsson, Andris Lipenitis, Master thesis, 2020
                 for now make Ignition crash?-->
             <!--         <inertia ixx="0.21" ixy="0.00" ixz="0.00" iyy="0.245" iyz="0.00" izz="0.245"/> -->
-            <inertia ixx="5.2539" ixy="0.0144" ixz="0.3341" iyy="7.9420" iyz="0.026" izz="6.9123"/>
-                <!-- Perfect rectangle -->
+            <inertia ixx="5.2539" ixy="0.0144" ixz="0.3341" iyy="7.9420" iyz="0.026" izz="6.9123" />
+            <!-- Perfect rectangle -->
             <!--        <inertia
             ixx="${mass/12*(y_size*y_size+z_size*z_size)}" ixy="0.0" ixz="0.0"
@@ -81,5 +83,5 @@
     </xacro:thruster>
     <xacro:if value="$(arg simulation)">
-        <xacro:include filename="$(find rov_description)/description/hydrodynamics.xacro"/>
+        <xacro:include filename="$(find rov_description)/description/hydrodynamics.xacro" />
         <gazebo>
             <plugin
@@ -93,17 +95,7 @@
                 <dimensions>3</dimensions>
                 <robot_base_frame>base_link</robot_base_frame>
-                <odom_publish_frequency>20</odom_publish_frequency>
-                <dimensions>3</dimensions>
-                <gaussian_noise>0.5</gaussian_noise>
+                <odom_publish_frequency>40</odom_publish_frequency>
+                <gaussian_noise>0.0004</gaussian_noise>
             </plugin>
-            <!-- If you want to publish world -> base_link transform -->
-            <!-- <plugin
-                filename="gz-sim-pose-publisher-system"
-                name="gz::sim::systems::PosePublisher">
-                <publish_link_pose>false</publish_link_pose>
-                <publish_collision_pose>false</publish_collision_pose>
-                <publish_visual_pose>false</publish_visual_pose>
-                <publish_nested_model_pose>true</publish_nested_model_pose>
-            </plugin> -->
         </gazebo>
     </xacro:if>

File: ros2_ws/src/rov/rov_description/description/sensors/camera.xacro (robot description, xacro)
@@ -6,4 +6,5 @@
         <parent link="chassis" />
         <child link="camera_base" />
+        <origin xyz="0.155 0 0" />
     </joint>
     <link name="camera">
@@ -27,7 +28,17 @@
     <xacro:if value="$(arg simulation)">
         <gazebo>
-            <plugin filename="gz-sim-joint-position-controller-system"
+            <plugin
+                filename="gz-sim-joint-position-controller-system"
                 name="gz::sim::systems::JointPositionController">
                 <joint_name>camera_joint</joint_name>
+                <topic>joint/knee_joint/0/cmd_pos</topic>
+                <p_gain>10.0</p_gain>
+                <i_gain>0.0</i_gain>
+                <d_gain>1.0</d_gain>
+                <i_max>100</i_max>
+                <i_min>-100</i_min>
+                <cmd_max>100</cmd_max>
+                <cmd_min>-100</cmd_min>
+                <cmd_offset>0.0</cmd_offset>
             </plugin>
         </gazebo>
@@ -47,4 +58,5 @@
                     </clip>
                 </camera>
+                <topic>/camera/image_raw</topic>
                 <always_on>1</always_on>
                 <update_rate>30</update_rate>

File: ros2_ws/src/rov/rov_description/description/sensors/depth_sensor.xacro (robot description, xacro)
@@ -1,4 +1,4 @@
 <?xml version="1.0"?>
-<robot xmlns:xacro="http://www.ros.org/wiki/xacro" >
+<robot xmlns:xacro="http://www.ros.org/wiki/xacro">
     <xacro:macro name="depth_sensor" params="name parent *origin">
         <link name="${name}">
@@ -9,7 +9,9 @@
             <child link="${name}" />
         </joint>
+        <!-- <xacro:if value="$(arg simulation)"> -->
+        <!-- </xacro:if> -->
     </xacro:macro>
     <xacro:depth_sensor name="Bar30" parent="chassis">
-        <origin xyz="0 0 0" rpy="0 0 0"/>
+        <origin xyz="0 0 0" rpy="0 0 0" />
     </xacro:depth_sensor>
 </robot>

File: ros2_ws/src/rov/rov_description/description/sensors/imu.xacro (robot description, xacro)
@@ -1,10 +1,10 @@
 <?xml version="1.0"?>
-<robot xmlns:xacro="http://www.ros.org/wiki/xacro" >
+<robot xmlns:xacro="http://www.ros.org/wiki/xacro">
     <xacro:macro name="imu" params="name parent *origin">
-        <link name="${name}"/>
+        <link name="${name}" />
         <joint name="{name}_joint" type="fixed">
-            <xacro:insert_block name="origin"/>
-            <parent link="${parent}"/>
-            <child link="${name}"/>
+            <xacro:insert_block name="origin" />
+            <parent link="${parent}" />
+            <child link="${name}" />
         </joint>
         <xacro:if value="$(arg simulation)">
@@ -21,33 +21,33 @@
                             <x>
                                 <noise type="gaussian">
-                                <mean>0</mean>
-                                <stddev>0.009</stddev>
-                                <bias_mean>0.00075</bias_mean>
-                                <bias_stddev>0.005</bias_stddev>
-                                <dynamic_bias_stddev>0.00002</dynamic_bias_stddev>
-                                <dynamic_bias_correlation_time>400.0</dynamic_bias_correlation_time>
-                                <precision>0.00025</precision>
+                                    <mean>0</mean>
+                                    <stddev>0.009</stddev>
+                                    <bias_mean>0.00075</bias_mean>
+                                    <bias_stddev>0.005</bias_stddev>
+                                    <dynamic_bias_stddev>0.00002</dynamic_bias_stddev>
+                                    <dynamic_bias_correlation_time>400.0</dynamic_bias_correlation_time>
+                                    <precision>0.00025</precision>
                                 </noise>
                             </x>
                             <y>
                                 <noise type="gaussian">
-                                <mean>0</mean>
-                                <stddev>0.009</stddev>
-                                <bias_mean>0.00075</bias_mean>
-                                <bias_stddev>0.005</bias_stddev>
-                                <dynamic_bias_stddev>0.00002</dynamic_bias_stddev>
-                                <dynamic_bias_correlation_time>400.0</dynamic_bias_correlation_time>
-                                <precision>0.00025</precision>
+                                    <mean>0</mean>
+                                    <stddev>0.009</stddev>
+                                    <bias_mean>0.00075</bias_mean>
+                                    <bias_stddev>0.005</bias_stddev>
+                                    <dynamic_bias_stddev>0.00002</dynamic_bias_stddev>
+                                    <dynamic_bias_correlation_time>400.0</dynamic_bias_correlation_time>
+                                    <precision>0.00025</precision>
                                 </noise>
                             </y>
                             <z>
                                 <noise type="gaussian">
-                                <mean>0</mean>
-                                <stddev>0.009</stddev>
-                                <bias_mean>0.00075</bias_mean>
-                                <bias_stddev>0.005</bias_stddev>
-                                <dynamic_bias_stddev>0.00002</dynamic_bias_stddev>
-                                <dynamic_bias_correlation_time>400.0</dynamic_bias_correlation_time>
-                                <precision>0.00025</precision>
+                                    <mean>0</mean>
+                                    <stddev>0.009</stddev>
+                                    <bias_mean>0.00075</bias_mean>
+                                    <bias_stddev>0.005</bias_stddev>
+                                    <dynamic_bias_stddev>0.00002</dynamic_bias_stddev>
+                                    <dynamic_bias_correlation_time>400.0</dynamic_bias_correlation_time>
+                                    <precision>0.00025</precision>
                                 </noise>
                             </z>
@@ -56,33 +56,33 @@
                             <x>
                                 <noise type="gaussian">
-                                <mean>0</mean>
-                                <stddev>0.021</stddev>
-                                <bias_mean>0.05</bias_mean>
-                                <bias_stddev>0.0075</bias_stddev>
-                                <dynamic_bias_stddev>0.000375</dynamic_bias_stddev>
-                                <dynamic_bias_correlation_time>175.0</dynamic_bias_correlation_time>
-                                <precision>0.005</precision>
+                                    <mean>0</mean>
+                                    <stddev>0.021</stddev>
+                                    <bias_mean>0.05</bias_mean>
+                                    <bias_stddev>0.0075</bias_stddev>
+                                    <dynamic_bias_stddev>0.000375</dynamic_bias_stddev>
+                                    <dynamic_bias_correlation_time>175.0</dynamic_bias_correlation_time>
+                                    <precision>0.005</precision>
                                 </noise>
                             </x>
                             <y>
                                 <noise type="gaussian">
-                                <mean>0</mean>
-                                <stddev>0.021</stddev>
-                                <bias_mean>0.05</bias_mean>
-                                <bias_stddev>0.0075</bias_stddev>
-                                <dynamic_bias_stddev>0.000375</dynamic_bias_stddev>
-                                <dynamic_bias_correlation_time>175.0</dynamic_bias_correlation_time>
-                                <precision>0.005</precision>
+                                    <mean>0</mean>
+                                    <stddev>0.021</stddev>
+                                    <bias_mean>0.05</bias_mean>
+                                    <bias_stddev>0.0075</bias_stddev>
+                                    <dynamic_bias_stddev>0.000375</dynamic_bias_stddev>
+                                    <dynamic_bias_correlation_time>175.0</dynamic_bias_correlation_time>
+                                    <precision>0.005</precision>
                                 </noise>
                             </y>
                             <z>
                                 <noise type="gaussian">
-                                <mean>0</mean>
-                                <stddev>0.021</stddev>
-                                <bias_mean>0.05</bias_mean>
-                                <bias_stddev>0.0075</bias_stddev>
-                                <dynamic_bias_stddev>0.000375</dynamic_bias_stddev>
-                                <dynamic_bias_correlation_time>175.0</dynamic_bias_correlation_time>
-                                <precision>0.005</precision>
+                                    <mean>0</mean>
+                                    <stddev>0.001</stddev>
+                                    <!-- <bias_mean>0.05</bias_mean> -->
+                                    <!-- <bias_stddev>0.0075</bias_stddev> -->
+                                    <!-- <dynamic_bias_stddev>0.000375</dynamic_bias_stddev> -->
+                                    <!-- <dynamic_bias_correlation_time>175.0</dynamic_bias_correlation_time> -->
+                                    <precision>0.005</precision>
                                 </noise>
                             </z>
@@ -97,5 +97,5 @@
     </xacro:macro>
     <xacro:imu name="imu" parent="chassis">
-        <origin xyz="0 0 0" rpy="0 0 0"/>
+        <origin xyz="0 0 0" rpy="0 0 0" />
     </xacro:imu>
 </robot>
